File: VU Switch/VU Switch.kicad_pcb (KiCad board)
At the start: 2 copper layers, 99.1 x 61.6 mm, 31 parts, among them J1 DC_12V, J10 VU_12V, J11 LED, J12 VU_5V, J13 VU_12V, J2 VU_12V, J3 SELECT, J4 INPUT4, J5 INPUT3, J6 INPUT2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

Commit message: Added license label
Other:
- board text added: "Licensed under CERN OHL v1.2"
